File: esp32-with-gsm.kicad_sch (KiCad schematic)
At the start: 17 parts, among them J1 LCD, J3 SPI Etx, J4 Buzzer, J5 Power in, U1 ESP32-DEVKITC-32D, U2 SIM800L-CORE

Commit message: updating circuit
Parts:
- removed J4: Buzzer, Connector_PinHeader_2.54mm:PinHeader_1x04_P2.54mm_Vertical, symbol Connector:Conn_01x04_Socket
- added BZ1: Buzzer, Buzzer_Beeper:Buzzer_12x9.5RM7.6, symbol Device:Buzzer
- added D4, D5, D6, D7: BAT54, Diode_SMD:D_1206_3216Metric_Pad1.42x1.75mm_HandSolder, symbol Diode:1N47xxA
- added J2: Bat Etx, Connector_PinHeader_2.54mm:PinHeader_1x08_P2.54mm_Vertical, symbol Connector:Conn_01x08_Socket
- added Q1: BC548, Package_TO_SOT_THT:TO-92_Inline, symbol Transistor_BJT:BC548
- added R10, R5, R6, R9: 560k, Resistor_SMD:R_0805_2012Metric, symbol Device:R_Small
- added R11, R7: 1K, Resistor_SMD:R_0805_2012Metric, symbol Device:R_Small
- added R12, R8: 560K, Resistor_SMD:R_0805_2012Metric, symbol Device:R_Small
- added R4: 1k, Resistor_SMD:R_0805_2012Metric, symbol Device:R_Small
Connections:
- net +3V3: now also D5.1 (K), D7.1 (K)
- net +5V: now also BZ1.1 (-), J2.1 (Pin_1); no longer J5.2 (Pin_2)
- net BUZZ: now also R4.1
- net GND: now also D4.2 (A), D6.2 (A), J2.2 (Pin_2), J2.4 (Pin_4), J2.5 (Pin_5), Q1.3 (E), R10.1, R12.2, R6.1, R8.2
- net ADC-P1: now reaches U1.J2-7 (IO32)
- net ADC-P1: now also R11.2, R12.1
- net ADC-P0: now reaches U1.J2-8 (IO33)
- net ADC-P0: now also R7.2, R8.1
- new net: D6.1 (K), D7.2 (A), R10.2, R11.1, R9.2
- new net: BZ1.2 (+), Q1.1 (C)
- new net: Q1.2 (B), R4.2
- new net: D4.1 (K), D5.2 (A), R5.2, R6.2, R7.1
- new net Vbat: J2.3 (Pin_3), R9.1
- new net Vin: J2.6 (Pin_6), J5.2 (Pin_2), R5.1

Commit message: Added v2r1
Parts:
- removed C1, C2: 1000uF, Capacitor_THT:C_Disc_D8.0mm_W2.5mm_P5.00mm, symbol Device:C_Small
- added DS1: WC1602A, Display:WC1602A, symbol Display_Character:WC1602A
- added Q2: BC548, Package_TO_SOT_THT:TO-92_Inline, symbol Transistor_BJT:BC548
- added R13, R14, R15, R16: 1k, Resistor_SMD:R_0805_2012Metric, symbol Device:R_Small
- D1, D2: footprint Diode_SMD:D_0805_2012Metric_Pad1.15x1.40mm_HandSolder -> Diode_SMD:D_0805_2012Metric
- D4, D5, D6, D7: footprint Diode_SMD:D_1206_3216Metric_Pad1.42x1.75mm_HandSolder -> Diode_SMD:D_0805_2012Metric
- U1: Description_1 (none) -> WiFi Development Tools (802.11) ESP32 General Development K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
Connections:
- net +5V: now also DS1.15 (LED(+)), DS1.2 (VDD), R15.2
- net BUZZ: now also U1.J3-16 (IO15); no longer U1.J3-14 (IO0)
- net GND: now also DS1.1 (VSS), Q2.3 (E), R16.1
- net LCD_DT4: now reaches U1.J2-17 (SD3)
- net LCD_DT4: now also DS1.10 (D3)
- net LCD_DT3: now reaches U1.J2-18 (CMD)
- net LCD_DT3: now also DS1.9 (D2)
- net LCD_EN: now reaches U1.J3-11 (IO17)
- net LCD_EN: now also DS1.6 (E)
- net LCD_RW: now reaches U1.J3-12 (IO16)
- net LCD_RW: now also DS1.5 (R/W)
- net LCD_RS: now reaches U1.J3-17 (SD1)
- net LCD_RS: now also DS1.4 (RS)
- net LCD_DT1: now reaches U1.J3-18 (SD0)
- net LCD_DT1: now also DS1.7 (D0)
- net LCD_DT2: now reaches U1.J3-19 (CLK)
- net LCD_DT2: now also DS1.8 (D1)
- new net: DS1.16 (LED(-)), R14.2
- new net: DS1.3 (VO), R15.1, R16.2
- new net: Q2.1 (C), R14.1
- new net: Q2.2 (B), R13.2
- new net LCD_BACKLIGHT: R13.1, U1.J3-14 (IO0)
